File: Hardware/Electronics/CCBucket/CCBucket.kicad_pcb (KiCad board)
At the start: 2 copper layers, 17 parts, among them J1 Conn_01x01, J2 Conn_01x01, J3 Conn_01x01, J4 Conn_01x01, J5 Conn_01x01, J6 Conn_01x01, J7 Conn_01x01, J8 Conn_01x01, J9 Conn_01x01, SW1 SW_SPDT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

Commit message: Added circuit board for bucket controller
Parts:
- C3: moved to F.Cu
- moved C3 10.2 mm to (163.1, 91.4)
- moved E1 0.13 mm to (168.9, 82.4)
Routing:
- net GND: track 45.0 -> 17.3 mm
- net +3V3: track 16.2 -> 9.05 mm
- added copper zone on B.Cu, net +3V3
- added copper zone on F.Cu, net +3V3
Other:
- board outline added: 18.3 x 32.5 mm
